File: OmegaGOTEK.kicad_pcb (KiCad board)
At the start: 2 copper layers, 424.2 x 99.1 mm, 75 parts, among them J3 Conn_01x02_Pin, J4 Conn_01x04_Pin, J5 Conn_01x02_Pin, J7 Conn_02x03_Counter_Clockwise, M0 Conn_01x02_Pin, P1 FLOPPY CONNECTOR, P2 PWR, P3 USB_A, Q1 MOFSET N DGS, Q2 MOFSET N DGS, Q3 MOFSET N DGS, Q4 MOFSET N DGS, Q5 MOFSET N DGS, Q6 MOFSET N DGS, U1 74HC04, U3 AT32F435RGT7, U4 AMS1117-3.3, U5 TM1651, U8 GD5F1GQ4UFYIGR, Y1 8 MHz

Commit message: More board work
Parts:
- added H5: MountingHole, MountingHole:MountingHole_2.2mm_M2_Pad_Via, F.Cu at (70.4, 48.3)
- added H6: MountingHole, MountingHole:MountingHole_2.2mm_M2_Pad_Via, F.Cu at (70.4, 27.9)
- added H7: MountingHole, MountingHole:MountingHole_2.2mm_M2_Pad_Via, F.Cu at (116.1, 27.9)
- added H8: MountingHole, MountingHole:MountingHole_2.2mm_M2_Pad_Via, F.Cu at (116.1, 48.3)
- C1: footprint Capacitor_SMD:C_0805_2012Metric_Pad1.18x1.45mm_HandSolder -> Capacitor_THT:CP_Radial_D5.0mm_P2.50mm
- U5: moved to B.Cu
- Y1: footprint Crystal:Crystal_HC49-U_Vertical -> Crystal:Crystal_HC49-4H_Vertical
- moved H4 442.7 mm to (71.7, 146.1)
- moved H3 441.1 mm to (71.7, 61.0)
- moved U3 293.1 mm to (144.1, 109.2)
- moved P1 290.3 mm to (212.6, 67.3)
- moved P2 290.3 mm to (215.2, 130.8)
- moved U8 258.2 mm to (160.6, 91.4)
- moved L3 188.1 mm to (76.7, 101.6), turned to -90 degrees
- moved L5 187.3 mm to (76.7, 109.2), turned to 90 degrees
- moved L4 185.5 mm to (76.7, 95.2), turned to -90 degrees
- moved H1 181.5 mm to (213.9, 146.1)
- moved H2 177.5 mm to (213.9, 61.0)
- moved S4 173.9 mm to (71.7, 74.3), turned to 90 degrees
- moved S3 163.3 mm to (71.7, 85.1), turned to 90 degrees
- moved C19 156.2 mm to (97.1, 106.7), turned to -90 degrees
- moved R21 141.2 mm to (84.4, 103.1), turned to 90 degrees
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Routing:
- net +5V: track 0.00 -> 264.6 mm, vias 0 -> 1
- net +3.3V: track 0.00 -> 260.5 mm, vias 0 -> 1
- net DISP_CLK: track 0.00 -> 136.0 mm, vias 0 -> 9
- net DISP_DIO: track 0.00 -> 111.3 mm, vias 0 -> 3
- net DSEL: track 0.00 -> 92.1 mm, vias 0 -> 2
- net /BTN_LEFT: track 0.00 -> 90.9 mm, vias 0 -> 1
- net /BTN_RIGHT: track 0.00 -> 88.4 mm, vias 0 -> 1
- net Net-(P3-D-): track 0.00 -> 71.5 mm
- net PIN4: track 0.00 -> 68.5 mm
- net J7_PIN2: track 0.00 -> 59.4 mm
- net NRST: track 0.00 -> 56.0 mm
- net JUMPER_JA: track 0.00 -> 54.8 mm, vias 0 -> 1
- net DS0: track 0.00 -> 46.6 mm
- net JUMPER_JC: track 0.00 -> 43.0 mm, vias 0 -> 1
- net DS1: track 0.00 -> 42.5 mm
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- added copper zone on B.Cu, net GND
- added copper zone on F.Cu, net GND
Other:
- board size 424.2 x 99.1 mm -> 149.9 x 124.5 mm
