File: OmegaGOTEK.kicad_sch (KiCad schematic)
At the start: 36 parts, among them J5 Conn_01x02_Pin, M0 Conn_01x02_Pin, P1 FLOPPY CONNECTOR, Q1 MOFSET N DGS, Q2 MOFSET N DGS, Q3 MOFSET N DGS, Q4 MOFSET N DGS, Q5 MOFSET N DGS, Q6 MOFSET N DGS, U1 74HC04, U1 STM32F105V8Tx

Commit message: More updates
Parts:
- removed U1: STM32F105V8Tx, Package_QFP:LQFP-100_14x14mm_P0.5mm, symbol MCU_ST_STM32F1:STM32F105V8Tx
- added C1: 100nF, symbol Device:C
- added J3, RST: Conn_01x02_Pin, symbol Connector:Conn_01x02_Pin
- added J4: Conn_01x04_Pin, symbol Connector:Conn_01x04_Pin
- added JP1: Conn_02x02_Top_Bottom, symbol Connector_Generic:Conn_02x02_Top_Bottom
- added LED1: SLR0403BRA1BD, SLR0403BRA1BD:LED-SEG-TH_SLR0403BRA1BD, symbol OmegaGOTEK_Library:SLR0403BRA1BD
- added U5: TM1651, TM1651:SOIC-16_L9.9-W3.9-P1.27-LS6.0-BL, symbol OmegaGOTEK_Library:TM1651
Connections:
- net +5V: now also J4.4 (Pin_4)
- net GND: now also C1.2, JP1.1 (Pin_1), RST.2 (Pin_2), U5.1 (GND)
- new net: LED1.8 (DIG3), U5.10 (GRID3)
- new net: LED1.9 (DIG2), U5.11 (GRID2)
- new net: LED1.12 (DIG1), U5.12 (GRID1)
- new net: LED1.11 (A), U5.2 (SEG1/K1)
- new net: LED1.7 (B), U5.3 (SEG2/K2)
- new net: LED1.4 (C), U5.4 (SEG3/K3)
- new net: LED1.2 (D), LED1.3 (DP), U5.5 (SEG4/K4)
- new net: LED1.1 (E), U5.6 (SEG5/K5)
- new net: LED1.10 (F), U5.7 (SEG6/K6)
- new net: LED1.5 (G), U5.8 (SEG7/K7)
- new net: LED1.6 (NC), U5.9 (GRID4)
- new net +3.3V: C1.1, J3.2 (Pin_2), JP1.2 (Pin_2), U5.13 (VDD)
- new net BOOT_0: J3.1 (Pin_1)
- new net CLK: JP1.3 (Pin_3), U5.15 (CLK)
- new net DIO: JP1.4 (Pin_4), U5.14 (DIO)
- new net JTCK-SWCLK: J4.3 (Pin_3)
- new net NRST: RST.1 (Pin_1)
- new net USART1_RX: J4.1 (Pin_1)
- new net USART1_TX: J4.2 (Pin_2)
- no-connect marks 2 -> 3
Other:
- note added: "FLOPPY CONNECTOR"
- note added: "LED DISPLAY BOARD"
- note added: "PRG PORT"
- moved on the sheet: C20, J5, JA, JB, JC, M0, P1, PU1, PU10, PU11, PU12, PU13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

Commit message: Finished schematic
Parts:
- added C16, C2, C23, C3, C4, C6, C7, C8, C9: 100nF, symbol Device:C
- added C19: 10µF, symbol Device:C_Polarized
- added C3, C5: 22pF, symbol Device:C
- added J7: Conn_02x03_Counter_Clockwise, Connector_PinHeader_2.54mm:PinHeader_2x03_P2.54mm_Horizontal, symbol Connector_Generic:Conn_02x03_Odd_Even
- added L3, L4, L5: LED, symbol Device:LED
- added P2: PWR, Connector_PinHeader_2.54mm:PinHeader_1x04_P2.54mm_Horizontal, symbol Connector_Generic:Conn_01x04
- added P3: USB_A, symbol Connector:USB_A
- added R1, R2: 22, symbol Device:R_US
- added R20, R21, R3: 1K, symbol Device:R_US
- added S3, S4: SW_MEC_5E, Button_Switch_THT:SW_Tactile_SKHH_Angled, symbol Switch:SW_Push
- added U3: AT32F435RGT7, OmegaGOTEK_Library:LQFP-64_L10.0-W10.0-P0.50-LS12.0-BL, symbol OmegaGOTEK_Library:AT32F435RGT7
- added U4: AMS1117-3.3, Package_TO_SOT_SMD:SOT-223-3_TabPin2, symbol Regulator_Linear:AMS1117-3.3
- added U8: GD5F1GQ4UFYIGR, OmegaGOTEK_Library:WSON-8_L8.0-W6.0-P1.27-TL-EP, symbol OmegaGOTEK_Library:GD5F1GQ4UFYIGR
- added Y1: 8 MHz, symbol Device:Crystal
- C1: symbol Device:C -> Device:C_Polarized
- JP1: footprint (none) -> Connector_PinHeader_2.54mm:PinHeader_2x02_P2.54mm_Horizontal
- LED1: footprint SLR0403BRA1BD:LED-SEG-TH_SLR0403BRA1BD -> OmegaGOTEK_Library:LED-SEG-TH_SLR0403BRA1BD
- U5: footprint TM1651:SOIC-16_L9.9-W3.9-P1.27-LS6.0-BL -> OmegaGOTEK_Library:SOIC-16_L9.9-W3.9-P1.27-LS6.0-BL
Connections:
- net +3.3V: now also C16.1, C2.1, C3.1, C6.1, C7.1, C8.1, C9.1, J7.6 (Pin_6), R20.1, R21.2, R3.2, U3.1 (VBAT), U3.13 (VDDA/VREF+), U3.19 (VDD), U3.32 (VDD), U3.48 (VDD), U3.64 (VDD), U4.2 (VO), U8.3 (~{WP}/SIO2), U8.7 (~{HOLD}/SIO3), U8.8 (VCC); no longer C1.1
- net +5V: now also C1.1, C19.1, C23.1, P2.1 (Pin_1), U4.3 (VI)
- net BOOT_0: now also U3.60 (BOOT0)
- net DIR: now also U3.26 (PB0)
- net DSEL: now also L4.2 (A), U3.14 (PA0)
- net DSKCHG: now also U3.59 (PB7)
- net GND: now also C16.2, C19.2, C2.2, C23.2, C3.1, C3.2, C4.2, C5.1, C6.2, C7.2, C8.2, C9.2, J7.5 (Pin_5), P2.2 (Pin_2), P2.3 (Pin_3), P3.4 (GND), P3.5 (Shield), S3.1, S4.1, U3.12 (VSSA/VREF-), U3.18 (VSS), U3.31 (PH3), U3.47 (PH2), U3.63 (VSS), U4.1 (GND), U8.4 (VSS), U8.9 (EP); no longer C1.2
- net INDEX: now also U3.61 (PB8)
- net JTCK-SWCLK: now also U3.49 (PA14)
- net JUMPER_JA: now also U3.37 (PC6)
- net JUMPER_JB: now also U3.16 (PA2)
- net JUMPER_JC: now also U3.27 (PB1)
- net NRST: now also C4.1, R3.1, U3.7 (NRST)
- net RDDATA: now also U3.23 (PA7)
- net READY: now also U3.55 (PB3)
- net SIDE: now also U3.56 (PB4)
- net STEP: now also U3.15 (PA1)
- net TRK00: now also U3.58 (PB6)
- net USART1_RX: now also U3.43 (PA10)
- net USART1_TX: now also U3.42 (PA9)
- net WDATA: now also U3.41 (PA8)
- net WGATE: now also U3.62 (PB9)
- net WPT: now also U3.57 (PB5)
- new net: C3.2, U3.5 (PH0), Y1.2
- new net: C5.2, U3.6 (PH1), Y1.1
- new net: L4.1 (K), R20.2
- new net: C1.2, P3.1 (VBUS)
- new net: P3.2 (D-), R2.1
- new net: P3.3 (D+), R1.1
- new net: L3.2 (A), L5.2 (A), R21.1
- new net BTN_LEFT: S4.2, U3.39 (PC8)
- new net BTN_RIGHT: S3.2, U3.38 (PC7)
- new net DISP_CLK: J7.3 (Pin_3), L3.1 (K), U3.30 (PB11)
- new net DISP_DIO: J7.4 (Pin_4), L5.1 (K), U3.29 (PB10)
- new net J7_PIN1: J7.1 (Pin_1), U3.51 (PC10)
- new net J7_PIN2: J7.2 (Pin_2), U3.52 (PC11)
- new net OTG_FS_DM: R2.2, U3.45 (PA12)
- new net OTG_FS_DP: R1.2, U3.44 (PA11)
- new net SPI_FLASH_CLK: U3.34 (PB13), U8.6 (SCLK)
- new net SPI_FLASH_CS: U3.33 (PB12), U8.1 (~{CS})
- new net SPI_FLASH_DI: U3.36 (PB15), U8.5 (SI/SIO0)
- new net SPI_FLASH_DO: U3.35 (PB14), U8.2 (SO/SIO1)
- no-connect marks 3 -> 23
Other:
- note added: "1"
- note added: "DISPLAY PORT"
- note added: "MICROPROCESSOR"
- note added: "POWER REGULATION"
- note added: "SPI FLASH"
- note added: "USB"
- title: (none) -> GOTEK FLOPPY EMULATOR
- moved on the sheet: C20, J3, J4, J5, JA, JB, JC, JP1, LED1, M0, P1, PU1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

Commit message: Started board design
Parts:
- added H1, H2, H3, H4: MountingHole, MountingHole:MountingHole_3.2mm_M3_Pad_Via, symbol Mechanical:MountingHole_Pad
- added unit 7 of U1
- C1, C16, C20, C23, C3, C4, C5, C6, C7, C8, C9: footprint (none) -> Capacitor_SMD:C_0805_2012Metric_Pad1.18x1.45mm_HandSolder
- C17: renamed from C2; footprint (none) -> Capacitor_SMD:C_0805_2012Metric_Pad1.18x1.45mm_HandSolder
- C18: renamed from C3; footprint (none) -> Capacitor_SMD:C_0805_2012Metric_Pad1.18x1.45mm_HandSolder
- C19: footprint (none) -> Capacitor_THT:CP_Radial_D5.0mm_P2.50mm
- J3, J5, M0, S0, S1: footprint (none) -> Connector_PinHeader_2.54mm:PinHeader_1x02_P2.54mm_Vertical
- J4: footprint (none) -> Connector_PinHeader_2.54mm:PinHeader_2x02_P2.54mm_Vertical
- JA1: renamed from JA; footprint (none) -> Connector_PinHeader_2.54mm:PinHeader_1x02_P2.54mm_Vertical
- JB1: renamed from JB; footprint (none) -> Connector_PinHeader_2.54mm:PinHeader_1x02_P2.54mm_Vertical
- JC1: renamed from JC; footprint (none) -> Connector_PinHeader_2.54mm:PinHeader_1x02_P2.54mm_Vertical
- L3, L4, L5: footprint (none) -> LED_THT:LED_D3.0mm
- P3: footprint (none) -> OmegaGOTEK_Library:USB-A-TH_676432911
- PU1, PU10, PU11, PU12, PU13, PU2, PU3, PU4, PU5, PU6, PU7, PU8, PU9, R1, R2, R20, R21, R3, RN1, RN3, RN4, RN5, RN6: footprint (none) -> Resistor_SMD:R_0805_2012Metric_Pad1.20x1.40mm_HandSolder
- Q1, Q2, Q3, Q4, Q5, Q6: footprint (none) -> Package_TO_SOT_SMD:SOT-23
- RN2: renamed from RN3; footprint (none) -> Resistor_SMD:R_0805_2012Metric_Pad1.20x1.40mm_HandSolder
- RST1: renamed from RST; footprint (none) -> Connector_PinHeader_2.54mm:PinHeader_1x02_P2.54mm_Vertical
- U1: footprint (none) -> Package_SO:SSOP-14_5.3x6.2mm_P0.65mm
- Y1: footprint (none) -> Crystal:Crystal_HC49-U_Vertical
Connections:
- net +5V: now also U1.7 (GND)
- net GND: now also H1.1, H2.1, H3.1, H4.1, U1.14 (VCC)
- no-connect marks 23 -> 21
Other:
- note added: "OPTIONAL FLASH FOR FAT12 IMAGE SUPPORT. NOT USED BY THE AMIGA FIRMWARE."
- note added: "PCB MOUNT HOLES"
- moved on the sheet: J7, L3, L5, R21

Commit message: More board work
Parts:
- added H5, H6, H7, H8: MountingHole, MountingHole:MountingHole_2.2mm_M2_Pad_Via, symbol Mechanical:MountingHole_Pad
- C1: footprint Capacitor_SMD:C_0805_2012Metric_Pad1.18x1.45mm_HandSolder -> Capacitor_THT:CP_Radial_D5.0mm_P2.50mm
- Y1: footprint Crystal:Crystal_HC49-U_Vertical -> Crystal:Crystal_HC49-4H_Vertical
Connections:
- net GND: now also H5.1, H6.1, H7.1, H8.1
Changed lines of the file:
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@@
   (junction (at 242.57 304.8) (diameter 0) (color 0 0 0 0)
   )
+  (junction (at 466.09 397.51) (diameter 0) (color 0 0 0 0)
+  )
   (junction (at 214.63 135.89) (diameter 0) (color 0 0 0 0)
   )
@@
   (junction (at 278.13 163.83) (diameter 0) (color 0 0 0 0)
   )
+  (junction (at 453.39 388.62) (diameter 0) (color 0 0 0 0)
+  )
   (junction (at 427.99 168.91) (diameter 0) (color 0 0 0 0)
   )
@@
   (junction (at 90.17 325.12) (diameter 0) (color 0 0 0 0)
   )
+  (junction (at 453.39 383.54) (diameter 0) (color 0 0 0 0)
+  )
   (junction (at 427.99 273.05) (diameter 0) (color 0 0 0 0)
   )
@@
   (junction (at 382.27 299.72) (diameter 0) (color 0 0 0 0)
   )
+  (junction (at 453.39 393.7) (diameter 0) (color 0 0 0 0)
+  )
   (junction (at 346.71 146.05) (diameter 0) (color 0 0 0 0)
   )
@@
     (stroke (width 0) (type default))
   )
+  (wire (pts (xy 466.09 397.51) (xy 466.09 398.78))
+    (stroke (width 0) (type default))
+  )
   (wire (pts (xy 144.78 72.39) (xy 144.78 69.85))
     (stroke (width 0) (type default))
@@
     (stroke (width 0) (type default))
   )
+  (wire (pts (xy 453.39 378.46) (xy 453.39 383.54))
+    (stroke (width 0) (type default))
+  )
   (wire (pts (xy 99.06 349.25) (xy 196.85 349.25))
     (stroke (width 0) (type default))
@@
     (stroke (width 0) (type default))
   )
+  (wire (pts (xy 450.85 383.54) (xy 453.39 383.54))
+    (stroke (width 0) (type default))
+  )
   (wire (pts (xy 424.18 97.79) (xy 431.8 97.79))
     (stroke (width 0) (type default))
@@
     (stroke (width 0) (type default))
   )
+  (wire (pts (xy 453.39 397.51) (xy 466.09 397.51))
+    (stroke (width 0) (type default))
+  )
   (wire (pts (xy 273.05 312.42) (xy 273.05 320.04))
     (stroke (width 0) (type default))
@@
     (stroke (width 0) (type default))
   )
+  (wire (pts (xy 450.85 393.7) (xy 453.39 393.7))
+    (stroke (width 0) (type default))
+  )
   (wire (pts (xy 498.475 231.14) (xy 498.475 213.36))
     (stroke (width 0) (type default))
@@
     (stroke (width 0) (type default))
   )
-  (wire (pts (xy 466.09 393.7) (xy 466.09 396.24))
-    (stroke (width 0) (type default))
-  )
   (wire (pts (xy 382.905 224.79) (xy 380.365 224.79))
     (stroke (width 0) (type default))
@@
     (stroke (width 0) (type default))
   )
+  (wire (pts (xy 450.85 378.46) (xy 453.39 378.46))
+    (stroke (width 0) (type default))
+  )
   (wire (pts (xy 400.05 146.05) (xy 400.05 140.97))
     (stroke (width 0) (type default))
@@
     (stroke (width 0) (type default))
   )
+  (wire (pts (xy 453.39 388.62) (xy 453.39 393.7))
+    (stroke (width 0) (type default))
+  )
   (wire (pts (xy 196.85 349.25) (xy 196.85 314.96))
     (stroke (width 0) (type default))
@@
     (stroke (width 0) (type default))
   )
+  (wire (pts (xy 453.39 383.54) (xy 453.39 388.62))
+    (stroke (width 0) (type default))
+  )
   (wire (pts (xy 471.805 228.6) (xy 474.98 228.6))
     (stroke (width 0) (type default))
@@
     (stroke (width 0) (type default))
   )
+  (wire (pts (xy 466.09 393.7) (xy 466.09 397.51))
+    (stroke (width 0) (type default))
+  )
   (wire (pts (xy 427.99 171.45) (xy 431.8 171.45))
     (stroke (width 0) (type default))
@@
     (stroke (width 0) (type default))
   )
+  (wire (pts (xy 453.39 393.7) (xy 453.39 397.51))
+    (stroke (width 0) (type default))
+  )
   (wire (pts (xy 427.99 173.99) (xy 363.22 173.99))
     (stroke (width 0) (type default))
@@
     (stroke (width 0) (type default))
   )
+  (wire (pts (xy 450.85 388.62) (xy 453.39 388.62))
+    (stroke (width 0) (type default))
+  )
   (wire (pts (xy 102.87 327.66) (xy 91.44 327.66))
     (stroke (width 0) (type default))
@@
     (stroke (width 0) (type default))
   )
-  (rectangle (start 453.39 374.65) (end 468.63 402.59)
+  (rectangle (start 440.69 374.65) (end 468.63 406.4)
     (stroke (width 0) (type dash))
     (fill (type none))
@@
     (effects (font (size 1.27 1.27)) (justify left bottom))
   )
-  (text "PCB MOUNT HOLES" (at 452.12 373.38 0)
+  (text "PCB MOUNT HOLES" (at 445.77 373.38 0)
     (effects (font (size 1.27 1.27)) (justify left bottom))
   )
@@
     )
   )
+  (symbol (lib_id "Mechanical:MountingHole_Pad") (at 448.31 393.7 90) (unit 1)
+    (in_bom yes) (on_board yes) (dnp no)
+    (property "Reference" "H8" (at 441.96 393.7 90)
+      (effects (font (size 1.27 1.27)) (justify right))
+    )
+    (property "Value" "MountingHole" (at 447.04 391.16 0)
+      (effects (font (size 1.27 1.27)) (justify left) hide)
+    )
+    (property "Footprint" "MountingHole:MountingHole_2.2mm_M2_Pad_Via" (at 448.31 393.7 0)
+      (effects (font (size 1.27 1.27)) hide)
+    )
+    (property "Datasheet" "~" (at 448.31 393.7 0)
+      (effects (font (size 1.27 1.27)) hide)
+    )
+    (pin "1")
+    (instances
+      (project "OmegaGOTEK"
+        (path "/1fd3d41e-a7ac-473b-adfc-4c72d1e05d19"
+          (reference "H8") (unit 1)
+        )
+      )
+    )
+  )
   (symbol (lib_id "Device:Q_NMOS_DGS") (at 142.24 264.16 0) (unit 1)
     (in_bom yes) (on_board yes) (dnp no) (fields_autoplaced)
@@
       (effects (font (size 1.27 1.27)) (justify right))
     )
-    (property "Footprint" "Crystal:Crystal_HC49-U_Vertical" (at 397.51 124.46 0)
+    (property "Footprint" "Crystal:Crystal_HC49-4H_Vertical" (at 397.51 124.46 0)
       (effects (font (size 1.27 1.27)) hide)
     )
@@
     )
   )
-  (symbol (lib_id "power:GND") (at 466.09 396.24 0) (unit 1)
+  (symbol (lib_id "power:GND") (at 466.09 398.78 0) (unit 1)
     (in_bom yes) (on_board yes) (dnp no) (fields_autoplaced)
-    (property "Reference" "#PWR034" (at 466.09 402.59 0)
+    (property "Reference" "#PWR034" (at 466.09 405.13 0)
       (effects (font (size 1.27 1.27)) hide)
     )
-    (property "Value" "GND" (at 466.09 401.32 0)
+    (property "Value" "GND" (at 466.09 403.86 0)
       (effects (font (size 1.27 1.27)))
     )
-    (property "Footprint" "" (at 466.09 396.24 0)
+    (property "Footprint" "" (at 466.09 398.78 0)
       (effects (font (size 1.27 1.27)) hide)
     )
-    (property "Datasheet" "" (at 466.09 396.24 0)
+    (property "Datasheet" "" (at 466.09 398.78 0)
       (effects (font (size 1.27 1.27)) hide)
     )
@@
     )
   )
+  (symbol (lib_id "Mechanical:MountingHole_Pad") (at 448.31 378.46 90) (unit 1)
+    (in_bom yes) (on_board yes) (dnp no)
+    (property "Reference" "H5" (at 441.96 378.46 90)
+      (effects (font (size 1.27 1.27)) (justify right))
+    )
+    (property "Value" "MountingHole" (at 447.04 375.92 0)
+      (effects (font (size 1.27 1.27)) (justify left) hide)
+    )
+    (property "Footprint" "MountingHole:MountingHole_2.2mm_M2_Pad_Via" (at 448.31 378.46 0)
+      (effects (font (size 1.27 1.27)) hide)
+    )
+    (property "Datasheet" "~" (at 448.31 378.46 0)
+      (effects (font (size 1.27 1.27)) hide)
+    )
+    (pin "1")
+    (instances
+      (project "OmegaGOTEK"
+        (path "/1fd3d41e-a7ac-473b-adfc-4c72d1e05d19"
+          (reference "H5") (unit 1)
+        )
+      )
+    )
+  )
   (symbol (lib_id "Device:R_US") (at 267.97 101.6 0) (unit 1)
     (in_bom yes) (on_board yes) (dnp no) (fields_autoplaced)
@@
     )
   )
+  (symbol (lib_id "Mechanical:MountingHole_Pad") (at 448.31 388.62 90) (unit 1)
+    (in_bom yes) (on_board yes) (dnp no)
+    (property "Reference" "H7" (at 441.96 388.62 90)
+      (effects (font (size 1.27 1.27)) (justify right))
+    )
+    (property "Value" "MountingHole" (at 447.04 386.08 0)
+      (effects (font (size 1.27 1.27)) (justify left) hide)
+    )
+    (property "Footprint" "MountingHole:MountingHole_2.2mm_M2_Pad_Via" (at 448.31 388.62 0)
+      (effects (font (size 1.27 1.27)) hide)
+    )
+    (property "Datasheet" "~" (at 448.31 388.62 0)
+      (effects (font (size 1.27 1.27)) hide)
+    )
+    (pin "1")
+    (instances
+      (project "OmegaGOTEK"
+        (path "/1fd3d41e-a7ac-473b-adfc-4c72d1e05d19"
+          (reference "H7") (unit 1)
+        )
+      )
+    )
+  )
   (symbol (lib_id "Device:R_US") (at 214.63 101.6 0) (unit 1)
     (in_bom yes) (on_board yes) (dnp no) (fields_autoplaced)
@@
     )
   )
+  (symbol (lib_id "Mechanical:MountingHole_Pad") (at 448.31 383.54 90) (unit 1)
+    (in_bom yes) (on_board yes) (dnp no)
+    (property "Reference" "H6" (at 441.96 383.54 90)
+      (effects (font (size 1.27 1.27)) (justify right))
+    )
+    (property "Value" "MountingHole" (at 447.04 381 0)
+      (effects (font (size 1.27 1.27)) (justify left) hide)
+    )
+    (property "Footprint" "MountingHole:MountingHole_2.2mm_M2_Pad_Via" (at 448.31 383.54 0)
+      (effects (font (size 1.27 1.27)) hide)
+    )
+    (property "Datasheet" "~" (at 448.31 383.54 0)
+      (effects (font (size 1.27 1.27)) hide)
+    )
+    (pin "1")
+    (instances
+      (project "OmegaGOTEK"
+        (path "/1fd3d41e-a7ac-473b-adfc-4c72d1e05d19"
+          (reference "H6") (unit 1)
+        )
+      )
+    )
+  )
   (symbol (lib_id "Switch:SW_Push") (at 369.57 102.87 0) (unit 1)
     (in_bom yes) (on_board yes) (dnp no)
@@
       (effects (font (size 1.27 1.27)) (justify left))
     )
-    (property "Footprint" "Capacitor_SMD:C_0805_2012Metric_Pad1.18x1.45mm_HandSolder" (at 336.2452 302.26 0)
+    (property "Footprint" "Capacitor_THT:CP_Radial_D5.0mm_P2.50mm" (at 336.2452 302.26 0)
       (effects (font (size 1.27 1.27)) hide)
     )
